Commit message: Fixed material colour issue that caused fingers to not appear in RVIZ

File: wsg_50_simulation/urdf/wsg_50.urdf.xacro (robot description, xacro)
@@ -83,7 +83,5 @@
 	     <!--box size="0.0175 0.03 0.024"/-->
           </geometry>
-          <material name="black">
-		<color rgba="0 0 0 0"/>
-      	  </material>
+          <material name="flat_black"/>
       </visual>
       <collision>
@@ -122,7 +120,5 @@
              <mesh filename="package://wsg_50_simulation/meshes/WSG-FMF.stl" scale="0.001 0.001 0.001"/>
           </geometry>
-          <material name="black">
-		<color rgba="0 0 0 0"/>
-      	  </material>
+          <material name="flat_black"/>
       </visual>
       <collision>
@@ -168,7 +164,5 @@
 	     <!--box size="0.0175 0.03 0.024"/-->
           </geometry>
-          <material name="black">
-		<color rgba="0 0 0 0"/>
-      	  </material>
+          <material name="flat_black"/>
       </visual>
       <collision>
@@ -207,7 +201,5 @@
              <mesh filename="package://wsg_50_simulation/meshes/WSG-FMF.stl" scale="0.001 0.001 0.001"/>
           </geometry>
-          <material name="black">
-		<color rgba="0 0 0 0"/>
-      	  </material>
+          <material name="flat_black"/>
       </visual>
       <collision>
